Commit message: Fix SLAM map smearing: DiffDrive plugin's configured wheel_separation (0.45, inherited from ROS1's skid-steer tuning) did not match this plugin's differential-drive kinematics, causing angular odometry to over-report rotation by ~50%. Empirically calibrated via controlled rotation tests (commanded angular velocity vs. Gazebo's actual reported yaw) to wheel_separation: 0.68, reducing error to ~1%. Also reverted an incorrect TF restructuring (base_link had been moved above body1 with the rotation applied at the wrong joint, re-introducing a frame mismatch) and tuned max_laser_range/minimum_travel_distance/minimum_travel_heading to match real sensor limits. Map now generates correctly, matching real environment geometry.

File: mobile_robot/urdf/mobile_robot.urdf (robot description, URDF)
Before this commit: robot mobile_robot, 9 links, 8 joints
Joints:
- removed joint body1_to_base_link
- removed joint dummy_to_body1
- added joint base_to_body1_link: type fixed, parent base_link, child body1, origin xyz=0 0 0 rpy=0 0 0
- added joint dummy_to_base: type fixed, parent dummy_root, child base_link, origin xyz=0 0 0 rpy=0 0 -1.5708

Commit message: Fix RViz2 robot model and Gazebo/RViz pose alignment; add Nav2 navigation
- RViz2: robot model now renders (RobotModel description from /robot_description topic, mesh package paths resolved after sourcing the workspace)
- Nav2: use dummy_root as base frame (body1 is rotated 90 deg from the real front), so RViz2 and Gazebo show the same position and heading
- AMCL: set initial pose from measured map->dummy_root transform (x=-1.001, y=3.032, yaw=1.593)
- Use sim time for Nav2 and RViz2; switch controller from MPPI to DWB
- README: remove resolved RViz2 limitation, add Nav2 and RViz2 setup sections

File: mobile_robot/urdf/mobile_robot.urdf (robot description, URDF)
Before this commit: robot mobile_robot, 9 links, 8 joints
Joints:
- removed joint base_to_body1_link
- removed joint dummy_to_base
- added joint body1_to_base_link: type fixed, parent body1, child base_link, origin xyz=0 0 0 rpy=0 0 -1.5708
- added joint dummy_to_body1: type fixed, parent dummy_root, child body1, origin xyz=0 0 0 rpy=0 0 0

Commit message: Nav2 navigation working end-to-end: add /clock bridge, tune costmaps for narrow doorway, fix base frame and initial pose; update README

File: mobile_robot/urdf/mobile_robot.urdf (robot description, URDF)
Before this commit: robot mobile_robot, 9 links, 8 joints
Joints:
- joint body1_to_base_link: origin xyz=0 0 0 rpy=0 0 -1.5708 -> xyz=0 0 0 rpy=0 0 0
- joint dummy_to_body1: origin xyz=0 0 0 rpy=0 0 0 -> xyz=0 0 0 rpy=0 0 -1.5708
